File: SparkleTilt/SparkleTilt.kicad_pcb (KiCad board)
At the start: 2 copper layers, 150.2 x 149.8 mm, 22 parts, among them J1 ICSP, J2 USB_C_Receptacle_USB2.0_16P, SW1 SW_SPST, U1 ATmega328P-A, U2 CH340N, Y1 16MHz

Commit message: GND Net Update
Routing:
- net GND: track 126.2 -> 77.2 mm, vias 14 -> 10
